Commit message: Added wheels and movement

File: install/exia_ground_description/share/exia_ground_description/urdf/exia_ground.urdf (robot description, URDF)
Before this commit: robot exia_ground, 2 links, 1 joints
Links:
- removed link world
- added link base_footprint
- added link front_left_wheel, mass 2.0; collision cylinder length=0.05 radius=0.1; visual cylinder length=0.05 radius=0.1
- added link front_right_wheel, mass 2.0; collision cylinder length=0.05 radius=0.1; visual cylinder length=0.05 radius=0.1
- added link rear_left_wheel, mass 2.0; collision cylinder length=0.05 radius=0.1; visual cylinder length=0.05 radius=0.1
- added link rear_right_wheel, mass 2.0; collision cylinder length=0.05 radius=0.1; visual cylinder length=0.05 radius=0.1
Joints:
- removed joint world_to_base
- added joint base_joint: type fixed, parent base_footprint, child base_link, origin xyz=0 0 0.2 rpy=0 0 0
- added joint front_left_wheel_joint: type continuous, parent base_link, child front_left_wheel, origin xyz=0.2 0.225 -0.1 rpy=0 0 0, axis 0 1 0
- added joint front_right_wheel_joint: type continuous, parent base_link, child front_right_wheel, origin xyz=0.2 -0.225 -0.1 rpy=0 0 0, axis 0 1 0
- added joint rear_left_wheel_joint: type continuous, parent base_link, child rear_left_wheel, origin xyz=-0.2 0.225 -0.1 rpy=0 0 0, axis 0 1 0
- added joint rear_right_wheel_joint: type continuous, parent base_link, child rear_right_wheel, origin xyz=-0.2 -0.225 -0.1 rpy=0 0 0, axis 0 1 0

Commit message: added imu sensor

File: install/exia_ground_description/share/exia_ground_description/urdf/exia_ground.urdf (robot description, URDF)
Before this commit: robot exia_ground, 6 links, 5 joints
Links:
- added link imu_link, mass 0.01; collision box size=0.025 0.025 0.01; visual box size=0.025 0.025 0.01
Joints:
- added joint imu_joint: type fixed, parent base_link, child imu_link, origin xyz=0 0 0.105 rpy=0 0 0
