Commit message: first iteration of pure pursuit working

File: install/exia_ground_description/share/exia_ground_description/urdf/exia_ground.urdf.xacro (robot description, xacro)
@@ -254,4 +254,43 @@
     <axis xyz="0 1 0"/>
     <dynamics damping="0.01" friction="0.0"/>
+  </joint>
+  <!-- ==================== BRAKE SYSTEM ==================== -->
+  <!-- Virtual brake actuator for simulation -->
+  <!-- In real hardware: This maps to a brake motor/servo/actuator -->
+  <!-- The brake_joint position (0-1) represents brake engagement level -->
+  <!-- 0 = no brake, 1 = full brake -->
+  <link name="brake_actuator_link">
+    <visual>
+      <origin xyz="0 0 0" rpy="0 0 0"/>
+      <geometry>
+        <box size="0.05 0.08 0.03"/>
+      </geometry>
+      <material name="red">
+        <color rgba="0.8 0.2 0.2 1"/>
+      </material>
+    </visual>
+    <collision>
+      <origin xyz="0 0 0" rpy="0 0 0"/>
+      <geometry>
+        <box size="0.05 0.08 0.03"/>
+      </geometry>
+    </collision>
+    <inertial>
+      <mass value="0.5"/>
+      <origin xyz="0 0 0" rpy="0 0 0"/>
+      <inertia ixx="0.0001" ixy="0" ixz="0"
+               iyy="0.0001" iyz="0"
+               izz="0.0001"/>
+    </inertial>
+  </link>
+  <!-- Brake actuator joint - position controlled (0.0 to 1.0) -->
+  <!-- This is a virtual joint for control purposes -->
+  <joint name="brake_joint" type="revolute">
+    <parent link="base_link"/>
+    <child link="brake_actuator_link"/>
+    <origin xyz="-0.15 0 -0.05" rpy="0 0 0"/>
+    <axis xyz="0 1 0"/>
+    <limit lower="0.0" upper="1.0" effort="1000.0" velocity="5.0"/>
+    <dynamics damping="0.1" friction="0.0"/>
   </joint>
   <!-- ==================== IMU SENSOR ==================== -->
@@ -384,4 +423,10 @@
       <state_interface name="velocity"/>
     </joint>
+    <!-- Brake joint - position control (0.0 to 1.0 engagement) -->
+    <joint name="brake_joint">
+      <command_interface name="position"/>
+      <state_interface name="position"/>
+      <state_interface name="velocity"/>
+    </joint>
   </ros2_control>
   <gazebo>
@@ -389,4 +434,5 @@
       <robot_param>robot_description</robot_param>
       <robot_param_node>robot_state_publisher</robot_param_node>
+      <!-- Only pass minimal hardware config - controllers loaded by spawners -->
       <parameters>$(arg config_path)</parameters>
     </plugin>

Commit message: updated udrf chassis for atv

File: install/exia_ground_description/share/exia_ground_description/urdf/exia_ground.urdf.xacro (robot description, xacro)
@@ -5,9 +5,9 @@
   <!-- ==================== PROPERTIES ==================== -->
   <!-- Chassis dimensions -->
-  <!-- Length: 0.6m, Width: 0.4m, Height: 0.2m -->
+  <!-- Length: 2.11m, Width: 1.2m, Height: 0.6m -->
   <!-- Wheel properties -->
-  <!-- Radius: 0.1m, Width: 0.05m -->
-  <!-- Wheel separation (Y): 0.45m (center to center) -->
-  <!-- Wheel base (X): 0.4m (front to rear axle) -->
+  <!-- Radius: 0.3m, Width: 0.15m -->
+  <!-- Track width (Y): 1.1m (wheel center to center) -->
+  <!-- Wheel base (X): 1.3m (front to rear axle) -->
   <!-- Drive type: Ackermann steering (car-like) -->
   <!-- Front wheels: steerable -->
@@ -21,5 +21,5 @@
       <origin xyz="0 0 0" rpy="0 0 0"/>
       <geometry>
-        <box size="0.6 0.4 0.2"/>
+        <box size="2.11 1.2 0.6"/>
       </geometry>
       <material name="blue">
@@ -30,22 +30,22 @@
       <origin xyz="0 0 0" rpy="0 0 0"/>
       <geometry>
-        <box size="0.6 0.4 0.2"/>
-      </geometry>
-    </collision>
-    <inertial>
-      <mass value="20.0"/>
+        <box size="2.11 1.2 0.6"/>
+      </geometry>
+    </collision>
+    <inertial>
+      <mass value="200.0"/>
       <origin xyz="0 0 0" rpy="0 0 0"/>
       <!-- Inertia for a box: Ixx = 1/12*m*(y^2+z^2), etc. -->
-      <inertia ixx="0.267" ixy="0" ixz="0"
-               iyy="0.667" iyz="0"
-               izz="0.867"/>
+      <inertia ixx="30.0" ixy="0" ixz="0"
+               iyy="80.2" iyz="0"
+               izz="98.2"/>
     </inertial>
   </link>
   <!-- Connect base_link to base_footprint -->
-  <!-- Elevate base_link by wheel_radius + half chassis height = 0.1 + 0.1 = 0.2m -->
+  <!-- Elevate base_link by wheel_radius + half chassis height = 0.3 + 0.3 = 0.6m -->
   <joint name="base_joint" type="fixed">
     <parent link="base_footprint"/>
     <child link="base_link"/>
-    <origin xyz="0 0 0.2" rpy="0 0 0"/>
+    <origin xyz="0 0 0.6" rpy="0 0 0"/>
   </joint>
   <!-- ==================== FRONT STEERING LINKS ==================== -->
@@ -56,5 +56,5 @@
       <origin xyz="0 0 0" rpy="0 0 0"/>
       <geometry>
-        <cylinder radius="0.02" length="0.03"/>
+        <cylinder radius="0.05" length="0.08"/>
       </geometry>
       <material name="grey">
@@ -65,13 +65,13 @@
       <origin xyz="0 0 0" rpy="0 0 0"/>
       <geometry>
-        <cylinder radius="0.02" length="0.03"/>
-      </geometry>
-    </collision>
-    <inertial>
-      <mass value="0.5"/>
-      <origin xyz="0 0 0" rpy="0 0 0"/>
-      <inertia ixx="0.0001" ixy="0" ixz="0"
-               iyy="0.0001" iyz="0"
-               izz="0.0001"/>
+        <cylinder radius="0.05" length="0.08"/>
+      </geometry>
+    </collision>
+    <inertial>
+      <mass value="2.0"/>
+      <origin xyz="0 0 0" rpy="0 0 0"/>
+      <inertia ixx="0.001" ixy="0" ixz="0"
+               iyy="0.001" iyz="0"
+               izz="0.001"/>
     </inertial>
   </link>
@@ -81,5 +81,5 @@
       <origin xyz="0 0 0" rpy="0 0 0"/>
       <geometry>
-        <cylinder radius="0.02" length="0.03"/>
+        <cylinder radius="0.05" length="0.08"/>
       </geometry>
       <material name="grey">
@@ -90,13 +90,13 @@
       <origin xyz="0 0 0" rpy="0 0 0"/>
       <geometry>
-        <cylinder radius="0.02" length="0.03"/>
-      </geometry>
-    </collision>
-    <inertial>
-      <mass value="0.5"/>
-      <origin xyz="0 0 0" rpy="0 0 0"/>
-      <inertia ixx="0.0001" ixy="0" ixz="0"
-               iyy="0.0001" iyz="0"
-               izz="0.0001"/>
+        <cylinder radius="0.05" length="0.08"/>
+      </geometry>
+    </collision>
+    <inertial>
+      <mass value="2.0"/>
+      <origin xyz="0 0 0" rpy="0 0 0"/>
+      <inertia ixx="0.001" ixy="0" ixz="0"
+               iyy="0.001" iyz="0"
+               izz="0.001"/>
     </inertial>
   </link>
@@ -107,7 +107,7 @@
     <parent link="base_link"/>
     <child link="front_left_steer_link"/>
-    <origin xyz="0.2 0.225 -0.1" rpy="0 0 0"/>
+    <origin xyz="0.65 0.55 -0.3" rpy="0 0 0"/>
     <axis xyz="0 0 1"/>
-    <limit lower="-0.6" upper="0.6" effort="1000.0" velocity="5.0"/>
+    <limit lower="-0.6" upper="0.6" effort="2000.0" velocity="3.0"/>
     <dynamics damping="0.0" friction="0.0"/>
   </joint>
@@ -116,7 +116,7 @@
     <parent link="base_link"/>
     <child link="front_right_steer_link"/>
-    <origin xyz="0.2 -0.225 -0.1" rpy="0 0 0"/>
+    <origin xyz="0.65 -0.55 -0.3" rpy="0 0 0"/>
     <axis xyz="0 0 1"/>
-    <limit lower="-0.6" upper="0.6" effort="1000.0" velocity="5.0"/>
+    <limit lower="-0.6" upper="0.6" effort="2000.0" velocity="3.0"/>
     <dynamics damping="0.0" friction="0.0"/>
   </joint>
@@ -128,5 +128,5 @@
       <origin xyz="0 0 0" rpy="1.5708 0 0"/>
       <geometry>
-        <cylinder radius="0.1" length="0.05"/>
+        <cylinder radius="0.3" length="0.15"/>
       </geometry>
       <material name="black">
@@ -137,13 +137,13 @@
       <origin xyz="0 0 0" rpy="1.5708 0 0"/>
       <geometry>
-        <cylinder radius="0.1" length="0.05"/>
-      </geometry>
-    </collision>
-    <inertial>
-      <mass value="2.0"/>
-      <origin xyz="0 0 0" rpy="1.5708 0 0"/>
-      <inertia ixx="0.00542" ixy="0" ixz="0"
-               iyy="0.00542" iyz="0"
-               izz="0.01"/>
+        <cylinder radius="0.3" length="0.15"/>
+      </geometry>
+    </collision>
+    <inertial>
+      <mass value="10.0"/>
+      <origin xyz="0 0 0" rpy="1.5708 0 0"/>
+      <inertia ixx="0.244" ixy="0" ixz="0"
+               iyy="0.244" iyz="0"
+               izz="0.45"/>
     </inertial>
   </link>
@@ -161,5 +161,5 @@
       <origin xyz="0 0 0" rpy="1.5708 0 0"/>
       <geometry>
-        <cylinder radius="0.1" length="0.05"/>
+        <cylinder radius="0.3" length="0.15"/>
       </geometry>
       <material name="black">
@@ -170,13 +170,13 @@
       <origin xyz="0 0 0" rpy="1.5708 0 0"/>
       <geometry>
-        <cylinder radius="0.1" length="0.05"/>
-      </geometry>
-    </collision>
-    <inertial>
-      <mass value="2.0"/>
-      <origin xyz="0 0 0" rpy="1.5708 0 0"/>
-      <inertia ixx="0.00542" ixy="0" ixz="0"
-               iyy="0.00542" iyz="0"
-               izz="0.01"/>
+        <cylinder radius="0.3" length="0.15"/>
+      </geometry>
+    </collision>
+    <inertial>
+      <mass value="10.0"/>
+      <origin xyz="0 0 0" rpy="1.5708 0 0"/>
+      <inertia ixx="0.244" ixy="0" ixz="0"
+               iyy="0.244" iyz="0"
+               izz="0.45"/>
     </inertial>
   </link>
@@ -196,5 +196,5 @@
       <origin xyz="0 0 0" rpy="1.5708 0 0"/>
       <geometry>
-        <cylinder radius="0.1" length="0.05"/>
+        <cylinder radius="0.3" length="0.15"/>
       </geometry>
       <material name="black">
@@ -205,13 +205,13 @@
       <origin xyz="0 0 0" rpy="1.5708 0 0"/>
       <geometry>
-        <cylinder radius="0.1" length="0.05"/>
-      </geometry>
-    </collision>
-    <inertial>
-      <mass value="2.0"/>
-      <origin xyz="0 0 0" rpy="1.5708 0 0"/>
-      <inertia ixx="0.00542" ixy="0" ixz="0"
-               iyy="0.00542" iyz="0"
-               izz="0.01"/>
+        <cylinder radius="0.3" length="0.15"/>
+      </geometry>
+    </collision>
+    <inertial>
+      <mass value="10.0"/>
+      <origin xyz="0 0 0" rpy="1.5708 0 0"/>
+      <inertia ixx="0.244" ixy="0" ixz="0"
+               iyy="0.244" iyz="0"
+               izz="0.45"/>
     </inertial>
   </link>
@@ -219,5 +219,5 @@
     <parent link="base_link"/>
     <child link="rear_left_wheel"/>
-    <origin xyz="-0.2 0.225 -0.1" rpy="0 0 0"/>
+    <origin xyz="-0.65 0.55 -0.3" rpy="0 0 0"/>
     <axis xyz="0 1 0"/>
     <dynamics damping="0.01" friction="0.0"/>
@@ -228,5 +228,5 @@
       <origin xyz="0 0 0" rpy="1.5708 0 0"/>
       <geometry>
-        <cylinder radius="0.1" length="0.05"/>
+        <cylinder radius="0.3" length="0.15"/>
       </geometry>
       <material name="black">
@@ -237,13 +237,13 @@
       <origin xyz="0 0 0" rpy="1.5708 0 0"/>
       <geometry>
-        <cylinder radius="0.1" length="0.05"/>
-      </geometry>
-    </collision>
-    <inertial>
-      <mass value="2.0"/>
-      <origin xyz="0 0 0" rpy="1.5708 0 0"/>
-      <inertia ixx="0.00542" ixy="0" ixz="0"
-               iyy="0.00542" iyz="0"
-               izz="0.01"/>
+        <cylinder radius="0.3" length="0.15"/>
+      </geometry>
+    </collision>
+    <inertial>
+      <mass value="10.0"/>
+      <origin xyz="0 0 0" rpy="1.5708 0 0"/>
+      <inertia ixx="0.244" ixy="0" ixz="0"
+               iyy="0.244" iyz="0"
+               izz="0.45"/>
     </inertial>
   </link>
@@ -251,5 +251,5 @@
     <parent link="base_link"/>
     <child link="rear_right_wheel"/>
-    <origin xyz="-0.2 -0.225 -0.1" rpy="0 0 0"/>
+    <origin xyz="-0.65 -0.55 -0.3" rpy="0 0 0"/>
     <axis xyz="0 1 0"/>
     <dynamics damping="0.01" friction="0.0"/>
@@ -264,5 +264,5 @@
       <origin xyz="0 0 0" rpy="0 0 0"/>
       <geometry>
-        <box size="0.05 0.08 0.03"/>
+        <box size="0.15 0.2 0.1"/>
       </geometry>
       <material name="red">
@@ -273,13 +273,13 @@
       <origin xyz="0 0 0" rpy="0 0 0"/>
       <geometry>
-        <box size="0.05 0.08 0.03"/>
-      </geometry>
-    </collision>
-    <inertial>
-      <mass value="0.5"/>
-      <origin xyz="0 0 0" rpy="0 0 0"/>
-      <inertia ixx="0.0001" ixy="0" ixz="0"
-               iyy="0.0001" iyz="0"
-               izz="0.0001"/>
+        <box size="0.15 0.2 0.1"/>
+      </geometry>
+    </collision>
+    <inertial>
+      <mass value="2.0"/>
+      <origin xyz="0 0 0" rpy="0 0 0"/>
+      <inertia ixx="0.001" ixy="0" ixz="0"
+               iyy="0.001" iyz="0"
+               izz="0.001"/>
     </inertial>
   </link>
@@ -289,7 +289,7 @@
     <parent link="base_link"/>
     <child link="brake_actuator_link"/>
-    <origin xyz="-0.15 0 -0.05" rpy="0 0 0"/>
+    <origin xyz="-0.5 0 -0.15" rpy="0 0 0"/>
     <axis xyz="0 1 0"/>
-    <limit lower="0.0" upper="1.0" effort="1000.0" velocity="5.0"/>
+    <limit lower="0.0" upper="1.0" effort="2000.0" velocity="5.0"/>
     <dynamics damping="0.1" friction="0.0"/>
   </joint>
@@ -301,5 +301,5 @@
       <origin xyz="0 0 0" rpy="0 0 0"/>
       <geometry>
-        <box size="0.025 0.025 0.01"/>
+        <box size="0.05 0.05 0.02"/>
       </geometry>
       <material name="green">
@@ -310,13 +310,13 @@
       <origin xyz="0 0 0" rpy="0 0 0"/>
       <geometry>
-        <box size="0.025 0.025 0.01"/>
-      </geometry>
-    </collision>
-    <inertial>
-      <mass value="0.01"/>
-      <origin xyz="0 0 0" rpy="0 0 0"/>
-      <inertia ixx="0.000001" ixy="0" ixz="0"
-               iyy="0.000001" iyz="0"
-               izz="0.000001"/>
+        <box size="0.05 0.05 0.02"/>
+      </geometry>
+    </collision>
+    <inertial>
+      <mass value="0.05"/>
+      <origin xyz="0 0 0" rpy="0 0 0"/>
+      <inertia ixx="0.00001" ixy="0" ixz="0"
+               iyy="0.00001" iyz="0"
+               izz="0.00001"/>
     </inertial>
   </link>
@@ -324,5 +324,5 @@
     <parent link="base_link"/>
     <child link="imu_link"/>
-    <origin xyz="0 0 0.105" rpy="0 0 0"/>
+    <origin xyz="0 0 0.31" rpy="0 0 0"/>
   </joint>
   <!-- ==================== GAZEBO FORTRESS PROPERTIES ==================== -->

Commit message: added lidar + imu integration

File: install/exia_ground_description/share/exia_ground_description/urdf/exia_ground.urdf.xacro (robot description, xacro)
@@ -326,4 +326,41 @@
     <origin xyz="0 0 0.31" rpy="0 0 0"/>
   </joint>
+  <!-- ==================== LIDAR SENSOR ==================== -->
+  <!-- 2D Lidar mounted on top of the chassis -->
+  <!-- Simulation: Gazebo Fortress GPU ray sensor -->
+  <!-- Hardware: Slamtec RPlidar S3 (40m range, 360 deg, 32000 samples/sec) -->
+  <!-- Mount position: Forward of center, above chassis for unobstructed 360 deg view -->
+  <link name="lidar_link">
+    <visual>
+      <origin xyz="0 0 0" rpy="0 0 0"/>
+      <geometry>
+        <!-- RPlidar S3 approximate dimensions: 76mm diameter, 41mm height -->
+        <cylinder radius="0.038" length="0.041"/>
+      </geometry>
+      <material name="dark_grey">
+        <color rgba="0.2 0.2 0.2 1"/>
+      </material>
+    </visual>
+    <collision>
+      <origin xyz="0 0 0" rpy="0 0 0"/>
+      <geometry>
+        <cylinder radius="0.038" length="0.041"/>
+      </geometry>
+    </collision>
+    <inertial>
+      <mass value="0.190"/>  <!-- RPlidar S3 weight: ~190g -->
+      <origin xyz="0 0 0" rpy="0 0 0"/>
+      <inertia ixx="0.00005" ixy="0" ixz="0"
+               iyy="0.00005" iyz="0"
+               izz="0.00007"/>
+    </inertial>
+  </link>
+  <!-- Lidar mount: Centered on chassis top, slightly forward -->
+  <!-- Z = 0.3 (half chassis height) + 0.02 (small clearance) + 0.02 (half lidar height) = 0.34m -->
+  <joint name="lidar_joint" type="fixed">
+    <parent link="base_link"/>
+    <child link="lidar_link"/>
+    <origin xyz="0.3 0 0.34" rpy="0 0 0"/>
+  </joint>
   <!-- ==================== GAZEBO FORTRESS PROPERTIES ==================== -->
   <!-- Wheel friction for traction -->
@@ -394,4 +431,36 @@
         </linear_acceleration>
       </imu>
+    </sensor>
+  </gazebo>
+  <!-- ==================== GAZEBO FORTRESS LIDAR SENSOR ==================== -->
+  <!-- 2D lidar sensor matching RPlidar S3 specifications -->
+  <!-- For hardware: Use rplidar_ros driver publishing to /scan topic -->
+  <gazebo reference="lidar_link">
+    <sensor name="gpu_lidar" type="gpu_lidar">
+      <update_rate>10</update_rate>
+      <topic>lidar</topic>
+      <gz_frame_id>lidar_link</gz_frame_id>
+      <lidar>
+        <scan>
+          <horizontal>
+            <samples>360</samples>
+            <resolution>1</resolution>
+            <min_angle>-3.14159</min_angle>
+            <max_angle>3.14159</max_angle>
+          </horizontal>
+          <vertical>
+            <samples>1</samples>
+            <resolution>1</resolution>
+            <min_angle>0</min_angle>
+            <max_angle>0</max_angle>
+          </vertical>
+        </scan>
+        <range>
+          <min>0.2</min>
+          <max>20.0</max>
+        </range>
+      </lidar>
+      <always_on>true</always_on>
+      <visualize>true</visualize>
     </sensor>
   </gazebo>

Commit message: basic functional SLAM and path-planning, config is setup but logic is still wrong

File: install/exia_ground_description/share/exia_ground_description/urdf/exia_ground.urdf.xacro (robot description, xacro)
@@ -356,10 +356,11 @@
     </inertial>
   </link>
-  <!-- Lidar mount: Centered on chassis top, slightly forward -->
-  <!-- Z = 0.3 (half chassis height) + 0.02 (small clearance) + 0.02 (half lidar height) = 0.34m -->
+  <!-- Lidar mount: Lower position to detect small obstacles -->
+  <!-- Z = 0.15m (15cm) to detect obstacles >= 15cm tall at close range -->
+  <!-- Tilted down 5 degrees (0.087 rad) to hit ground at ~1.7m distance -->
   <joint name="lidar_joint" type="fixed">
     <parent link="base_link"/>
     <child link="lidar_link"/>
-    <origin xyz="0.3 0 0.34" rpy="0 0 0"/>
+    <origin xyz="0.3 0 0.15" rpy="0 0.087 0"/>
   </joint>
   <!-- ==================== GAZEBO FORTRESS PROPERTIES ==================== -->

Commit message: pre revamp

File: install/exia_ground_description/share/exia_ground_description/urdf/exia_ground.urdf.xacro (robot description, xacro)
@@ -356,11 +356,11 @@
     </inertial>
   </link>
-  <!-- Lidar mount: Lower position to detect small obstacles -->
-  <!-- Z = 0.15m (15cm) to detect obstacles >= 15cm tall at close range -->
-  <!-- Tilted down 5 degrees (0.087 rad) to hit ground at ~1.7m distance -->
+  <!-- Lidar mount: Horizontal for accurate obstacle detection -->
+  <!-- Z = 0.35m (35cm above base_link) for good ground clearance -->
+  <!-- No tilt to avoid false ground detections in costmap -->
   <joint name="lidar_joint" type="fixed">
     <parent link="base_link"/>
     <child link="lidar_link"/>
-    <origin xyz="0.3 0 0.15" rpy="0 0.087 0"/>
+    <origin xyz="0.3 0 0.35" rpy="0 0 0"/>
   </joint>
   <!-- ==================== GAZEBO FORTRESS PROPERTIES ==================== -->
