Commit message: architecture revamp

File: install/exia_ground_description/share/exia_ground_description/urdf/exia_ground.urdf.xacro (robot description, xacro)
@@ -1 +1,579 @@
-/home/zech/exia_ws/src/exia_ground_description/urdf/exia_ground.urdf.xacro
+<?xml version="1.0"?>
+<robot name="exia_ground" xmlns:xacro="http://www.ros.org/wiki/xacro">
+  <!-- Xacro arguments -->
+  <xacro:arg name="config_path" default=""/>
+  <!-- ==================== PROPERTIES ==================== -->
+  <!-- Chassis dimensions -->
+  <!-- Length: 2.11m, Width: 1.2m, Height: 0.6m -->
+  <!-- Wheel properties -->
+  <!-- Radius: 0.3m, Width: 0.15m -->
+  <!-- Track width (Y): 1.1m (wheel center to center) -->
+  <!-- Wheel base (X): 1.3m (front to rear axle) -->
+  <!-- Drive type: Ackermann steering (car-like) -->
+  <!-- Front wheels: steerable -->
+  <!-- Rear wheels: driven -->
+  <!-- ==================== BASE FOOTPRINT ==================== -->
+  <!-- Ground projection of the robot - used for navigation -->
+  <link name="base_footprint"/>
+  <!-- ==================== BASE LINK (CHASSIS) ==================== -->
+  <link name="base_link">
+    <visual>
+      <origin xyz="0 0 0" rpy="0 0 0"/>
+      <geometry>
+        <box size="2.11 1.2 0.6"/>
+      </geometry>
+      <material name="blue">
+        <color rgba="0.2 0.2 0.8 1"/>
+      </material>
+    </visual>
+    <collision>
+      <origin xyz="0 0 0" rpy="0 0 0"/>
+      <geometry>
+        <box size="2.11 1.2 0.6"/>
+      </geometry>
+    </collision>
+    <inertial>
+      <mass value="200.0"/>
+      <origin xyz="0 0 0" rpy="0 0 0"/>
+      <!-- Inertia for a box: Ixx = 1/12*m*(y^2+z^2), etc. -->
+      <inertia ixx="30.0" ixy="0" ixz="0"
+               iyy="80.2" iyz="0"
+               izz="98.2"/>
+    </inertial>
+  </link>
+  <!-- Connect base_link to base_footprint -->
+  <!-- Elevate base_link by wheel_radius + half chassis height = 0.3 + 0.3 = 0.6m -->
+  <joint name="base_joint" type="fixed">
+    <parent link="base_footprint"/>
+    <child link="base_link"/>
+    <origin xyz="0 0 0.6" rpy="0 0 0"/>
+  </joint>
+  <!-- ==================== FRONT STEERING LINKS ==================== -->
+  <!-- These are the steering knuckles that rotate to steer the front wheels -->
+  <!-- FRONT LEFT STEERING LINK -->
+  <link name="front_left_steer_link">
+    <visual>
+      <origin xyz="0 0 0" rpy="0 0 0"/>
+      <geometry>
+        <cylinder radius="0.05" length="0.08"/>
+      </geometry>
+      <material name="grey">
+        <color rgba="0.5 0.5 0.5 1"/>
+      </material>
+    </visual>
+    <collision>
+      <origin xyz="0 0 0" rpy="0 0 0"/>
+      <geometry>
+        <cylinder radius="0.05" length="0.08"/>
+      </geometry>
+    </collision>
+    <inertial>
+      <mass value="2.0"/>
+      <origin xyz="0 0 0" rpy="0 0 0"/>
+      <inertia ixx="0.001" ixy="0" ixz="0"
+               iyy="0.001" iyz="0"
+               izz="0.001"/>
+    </inertial>
+  </link>
+  <!-- FRONT RIGHT STEERING LINK -->
+  <link name="front_right_steer_link">
+    <visual>
+      <origin xyz="0 0 0" rpy="0 0 0"/>
+      <geometry>
+        <cylinder radius="0.05" length="0.08"/>
+      </geometry>
+      <material name="grey">
+        <color rgba="0.5 0.5 0.5 1"/>
+      </material>
+    </visual>
+    <collision>
+      <origin xyz="0 0 0" rpy="0 0 0"/>
+      <geometry>
+        <cylinder radius="0.05" length="0.08"/>
+      </geometry>
+    </collision>
+    <inertial>
+      <mass value="2.0"/>
+      <origin xyz="0 0 0" rpy="0 0 0"/>
+      <inertia ixx="0.001" ixy="0" ixz="0"
+               iyy="0.001" iyz="0"
+               izz="0.001"/>
+    </inertial>
+  </link>
+  <!-- ==================== FRONT STEERING JOINTS ==================== -->
+  <!-- Revolute joints that allow front wheels to steer (rotate about Z axis) -->
+  <!-- FRONT LEFT STEERING JOINT -->
+  <joint name="front_left_steer_joint" type="revolute">
+    <parent link="base_link"/>
+    <child link="front_left_steer_link"/>
+    <origin xyz="0.65 0.55 -0.3" rpy="0 0 0"/>
+    <axis xyz="0 0 1"/>
+    <limit lower="-0.6" upper="0.6" effort="2000.0" velocity="3.0"/>
+    <dynamics damping="0.0" friction="0.0"/>
+  </joint>
+  <!-- FRONT RIGHT STEERING JOINT -->
+  <joint name="front_right_steer_joint" type="revolute">
+    <parent link="base_link"/>
+    <child link="front_right_steer_link"/>
+    <origin xyz="0.65 -0.55 -0.3" rpy="0 0 0"/>
+    <axis xyz="0 0 1"/>
+    <limit lower="-0.6" upper="0.6" effort="2000.0" velocity="3.0"/>
+    <dynamics damping="0.0" friction="0.0"/>
+  </joint>
+  <!-- ==================== FRONT WHEELS ==================== -->
+  <!-- Front wheels are children of steering links, allowing them to steer -->
+  <!-- FRONT LEFT WHEEL -->
+  <link name="front_left_wheel">
+    <visual>
+      <origin xyz="0 0 0" rpy="1.5708 0 0"/>
+      <geometry>
+        <cylinder radius="0.3" length="0.15"/>
+      </geometry>
+      <material name="black">
+        <color rgba="0.1 0.1 0.1 1"/>
+      </material>
+    </visual>
+    <collision>
+      <origin xyz="0 0 0" rpy="1.5708 0 0"/>
+      <geometry>
+        <cylinder radius="0.3" length="0.15"/>
+      </geometry>
+    </collision>
+    <inertial>
+      <mass value="10.0"/>
+      <origin xyz="0 0 0" rpy="1.5708 0 0"/>
+      <inertia ixx="0.244" ixy="0" ixz="0"
+               iyy="0.244" iyz="0"
+               izz="0.45"/>
+    </inertial>
+  </link>
+  <!-- Front left wheel joint - child of steering link -->
+  <joint name="front_left_wheel_joint" type="continuous">
+    <parent link="front_left_steer_link"/>
+    <child link="front_left_wheel"/>
+    <origin xyz="0 0 0" rpy="0 0 0"/>
+    <axis xyz="0 1 0"/>
+    <dynamics damping="0.1" friction="0.1"/>
+  </joint>
+  <!-- FRONT RIGHT WHEEL -->
+  <link name="front_right_wheel">
+    <visual>
+      <origin xyz="0 0 0" rpy="1.5708 0 0"/>
+      <geometry>
+        <cylinder radius="0.3" length="0.15"/>
+      </geometry>
+      <material name="black">
+        <color rgba="0.1 0.1 0.1 1"/>
+      </material>
+    </visual>
+    <collision>
+      <origin xyz="0 0 0" rpy="1.5708 0 0"/>
+      <geometry>
+        <cylinder radius="0.3" length="0.15"/>
+      </geometry>
+    </collision>
+    <inertial>
+      <mass value="10.0"/>
+      <origin xyz="0 0 0" rpy="1.5708 0 0"/>
+      <inertia ixx="0.244" ixy="0" ixz="0"
+               iyy="0.244" iyz="0"
+               izz="0.45"/>
+    </inertial>
+  </link>
+  <!-- Front right wheel joint - child of steering link -->
+  <joint name="front_right_wheel_joint" type="continuous">
+    <parent link="front_right_steer_link"/>
+    <child link="front_right_wheel"/>
+    <origin xyz="0 0 0" rpy="0 0 0"/>
+    <axis xyz="0 1 0"/>
+    <dynamics damping="0.1" friction="0.1"/>
+  </joint>
+  <!-- ==================== REAR WHEELS (DRIVE WHEELS) ==================== -->
+  <!-- Rear wheels are directly connected to base_link and provide propulsion -->
+  <!-- REAR LEFT WHEEL -->
+  <link name="rear_left_wheel">
+    <visual>
+      <origin xyz="0 0 0" rpy="1.5708 0 0"/>
+      <geometry>
+        <cylinder radius="0.3" length="0.15"/>
+      </geometry>
+      <material name="black">
+        <color rgba="0.1 0.1 0.1 1"/>
+      </material>
+    </visual>
+    <collision>
+      <origin xyz="0 0 0" rpy="1.5708 0 0"/>
+      <geometry>
+        <cylinder radius="0.3" length="0.15"/>
+      </geometry>
+    </collision>
+    <inertial>
+      <mass value="10.0"/>
+      <origin xyz="0 0 0" rpy="1.5708 0 0"/>
+      <inertia ixx="0.244" ixy="0" ixz="0"
+               iyy="0.244" iyz="0"
+               izz="0.45"/>
+    </inertial>
+  </link>
+  <joint name="rear_left_wheel_joint" type="continuous">
+    <parent link="base_link"/>
+    <child link="rear_left_wheel"/>
+    <origin xyz="-0.65 0.55 -0.3" rpy="0 0 0"/>
+    <axis xyz="0 1 0"/>
+    <dynamics damping="0.01" friction="0.0"/>
+  </joint>
+  <!-- REAR RIGHT WHEEL -->
+  <link name="rear_right_wheel">
+    <visual>
+      <origin xyz="0 0 0" rpy="1.5708 0 0"/>
+      <geometry>
+        <cylinder radius="0.3" length="0.15"/>
+      </geometry>
+      <material name="black">
+        <color rgba="0.1 0.1 0.1 1"/>
+      </material>
+    </visual>
+    <collision>
+      <origin xyz="0 0 0" rpy="1.5708 0 0"/>
+      <geometry>
+        <cylinder radius="0.3" length="0.15"/>
+      </geometry>
+    </collision>
+    <inertial>
+      <mass value="10.0"/>
+      <origin xyz="0 0 0" rpy="1.5708 0 0"/>
+      <inertia ixx="0.244" ixy="0" ixz="0"
+               iyy="0.244" iyz="0"
+               izz="0.45"/>
+    </inertial>
+  </link>
+  <joint name="rear_right_wheel_joint" type="continuous">
+    <parent link="base_link"/>
+    <child link="rear_right_wheel"/>
+    <origin xyz="-0.65 -0.55 -0.3" rpy="0 0 0"/>
+    <axis xyz="0 1 0"/>
+    <dynamics damping="0.01" friction="0.0"/>
+  </joint>
+  <!-- ==================== BRAKE SYSTEM ==================== -->
+  <!-- Virtual brake actuator for simulation -->
+  <!-- In real hardware: This maps to a brake motor/servo/actuator -->
+  <!-- The brake_joint position (0-1) represents brake engagement level -->
+  <!-- 0 = no brake, 1 = full brake -->
+  <link name="brake_actuator_link">
+    <visual>
+      <origin xyz="0 0 0" rpy="0 0 0"/>
+      <geometry>
+        <box size="0.15 0.2 0.1"/>
+      </geometry>
+      <material name="red">
+        <color rgba="0.8 0.2 0.2 1"/>
+      </material>
+    </visual>
+    <collision>
+      <origin xyz="0 0 0" rpy="0 0 0"/>
+      <geometry>
+        <box size="0.15 0.2 0.1"/>
+      </geometry>
+    </collision>
+    <inertial>
+      <mass value="2.0"/>
+      <origin xyz="0 0 0" rpy="0 0 0"/>
+      <inertia ixx="0.001" ixy="0" ixz="0"
+               iyy="0.001" iyz="0"
+               izz="0.001"/>
+    </inertial>
+  </link>
+  <!-- Brake actuator joint - position controlled (0.0 to 1.0) -->
+  <!-- This is a virtual joint for control purposes -->
+  <joint name="brake_joint" type="revolute">
+    <parent link="base_link"/>
+    <child link="brake_actuator_link"/>
+    <origin xyz="-0.5 0 -0.15" rpy="0 0 0"/>
+    <axis xyz="0 1 0"/>
+    <limit lower="0.0" upper="1.0" effort="2000.0" velocity="5.0"/>
+    <dynamics damping="0.1" friction="0.0"/>
+  </joint>
+  <!-- ==================== IMU SENSOR ==================== -->
+  <!-- IMU mounted on top of the chassis, centered -->
+  <!-- This represents the Yahboom 10-axis IMU for hardware deployment -->
+  <link name="imu_link">
+    <visual>
+      <origin xyz="0 0 0" rpy="0 0 0"/>
+      <geometry>
+        <box size="0.05 0.05 0.02"/>
+      </geometry>
+      <material name="green">
+        <color rgba="0.2 0.8 0.2 1"/>
+      </material>
+    </visual>
+    <collision>
+      <origin xyz="0 0 0" rpy="0 0 0"/>
+      <geometry>
+        <box size="0.05 0.05 0.02"/>
+      </geometry>
+    </collision>
+    <inertial>
+      <mass value="0.05"/>
+      <origin xyz="0 0 0" rpy="0 0 0"/>
+      <inertia ixx="0.00001" ixy="0" ixz="0"
+               iyy="0.00001" iyz="0"
+               izz="0.00001"/>
+    </inertial>
+  </link>
+  <joint name="imu_joint" type="fixed">
+    <parent link="base_link"/>
+    <child link="imu_link"/>
+    <origin xyz="0 0 0.31" rpy="0 0 0"/>
+  </joint>
+  <!-- ==================== LIDAR SENSOR ==================== -->
+  <!-- 2D Lidar mounted on top of the chassis -->
+  <!-- Simulation: Gazebo Fortress GPU ray sensor -->
+  <!-- Hardware: Slamtec RPlidar S3 (40m range, 360 deg, 32000 samples/sec) -->
+  <!-- Mount position: Forward of center, above chassis for unobstructed 360 deg view -->
+  <link name="lidar_link">
+    <visual>
+      <origin xyz="0 0 0" rpy="0 0 0"/>
+      <geometry>
+        <!-- RPlidar S3 approximate dimensions: 76mm diameter, 41mm height -->
+        <cylinder radius="0.038" length="0.041"/>
+      </geometry>
+      <material name="dark_grey">
+        <color rgba="0.2 0.2 0.2 1"/>
+      </material>
+    </visual>
+    <collision>
+      <origin xyz="0 0 0" rpy="0 0 0"/>
+      <geometry>
+        <cylinder radius="0.038" length="0.041"/>
+      </geometry>
+    </collision>
+    <inertial>
+      <mass value="0.190"/>  <!-- RPlidar S3 weight: ~190g -->
+      <origin xyz="0 0 0" rpy="0 0 0"/>
+      <inertia ixx="0.00005" ixy="0" ixz="0"
+               iyy="0.00005" iyz="0"
+               izz="0.00007"/>
+    </inertial>
+  </link>
+  <!-- Lidar mount: Horizontal for accurate obstacle detection -->
+  <!-- Z = 0.35m (35cm above base_link) for good ground clearance -->
+  <!-- No tilt to avoid false ground detections in costmap -->
+  <joint name="lidar_joint" type="fixed">
+    <parent link="base_link"/>
+    <child link="lidar_link"/>
+    <origin xyz="0.3 0 0.35" rpy="0 0 0"/>
+  </joint>
+  <!-- ==================== 3D LIDAR SENSOR ==================== -->
+  <!-- 360-degree 3D lidar for visualization (VLP-16 style) -->
+  <!-- NOT used for navigation - visualization only -->
+  <!-- Mounted above 2D lidar for full 360-degree 3D coverage -->
+  <link name="lidar_3d_link">
+    <visual>
+      <origin xyz="0 0 0" rpy="0 0 0"/>
+      <geometry>
+        <cylinder radius="0.05" length="0.07"/>
+      </geometry>
+      <material name="dark_grey">
+        <color rgba="0.2 0.2 0.2 1"/>
+      </material>
+    </visual>
+    <collision>
+      <origin xyz="0 0 0" rpy="0 0 0"/>
+      <geometry>
+        <cylinder radius="0.05" length="0.07"/>
+      </geometry>
+    </collision>
+    <inertial>
+      <mass value="0.83"/>
+      <origin xyz="0 0 0" rpy="0 0 0"/>
+      <inertia ixx="0.0005" ixy="0" ixz="0"
+               iyy="0.0005" iyz="0"
+               izz="0.001"/>
+    </inertial>
+  </link>
+  <joint name="lidar_3d_joint" type="fixed">
+    <parent link="base_link"/>
+    <child link="lidar_3d_link"/>
+    <origin xyz="0.3 0 0.42" rpy="0 0 0"/>
+  </joint>
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