Commit message: path planning fixed with 3D Lidar

File: src/exia_bringup/urdf/exia_ground.urdf.xacro (robot description, xacro)
@@ -2,4 +2,11 @@
 <robot name="exia_ground" xmlns:xacro="http://www.ros.org/wiki/xacro">
   <xacro:arg name="config_path" default=""/>
+  <xacro:arg name="lidar_horizontal_samples" default="360"/>
+  <xacro:arg name="lidar_vertical_samples" default="16"/>
+  <xacro:arg name="lidar_vertical_fov_min" default="-0.261799"/>
+  <xacro:arg name="lidar_vertical_fov_max" default="0.261799"/>
+  <xacro:arg name="lidar_range_min" default="1.5"/>
+  <xacro:arg name="lidar_range_max" default="20.0"/>
+  <xacro:arg name="lidar_update_rate" default="10"/>
   <link name="base_footprint"/>
   <link name="base_link">
@@ -285,33 +292,4 @@
       <origin xyz="0 0 0" rpy="0 0 0"/>
       <geometry>
-        <cylinder radius="0.038" length="0.041"/>
-      </geometry>
-      <material name="dark_grey">
-        <color rgba="0.2 0.2 0.2 1"/>
-      </material>
-    </visual>
-    <collision>
-      <origin xyz="0 0 0" rpy="0 0 0"/>
-      <geometry>
-        <cylinder radius="0.038" length="0.041"/>
-      </geometry>
-    </collision>
-    <inertial>
-      <mass value="0.190"/>
-      <origin xyz="0 0 0" rpy="0 0 0"/>
-      <inertia ixx="0.00005" ixy="0" ixz="0"
-               iyy="0.00005" iyz="0"
-               izz="0.00007"/>
-    </inertial>
-  </link>
-  <joint name="lidar_joint" type="fixed">
-    <parent link="base_link"/>
-    <child link="lidar_link"/>
-    <origin xyz="0.3 0 0.35" rpy="0 0 0"/>
-  </joint>
-  <link name="lidar_3d_link">
-    <visual>
-      <origin xyz="0 0 0" rpy="0 0 0"/>
-      <geometry>
         <cylinder radius="0.05" length="0.07"/>
       </geometry>
@@ -334,7 +312,7 @@
     </inertial>
   </link>
-  <joint name="lidar_3d_joint" type="fixed">
-    <parent link="base_link"/>
-    <child link="lidar_3d_link"/>
+  <joint name="lidar_joint" type="fixed">
+    <parent link="base_link"/>
+    <child link="lidar_link"/>
     <origin xyz="0.3 0 0.42" rpy="0 0 0"/>
   </joint>
@@ -407,12 +385,13 @@
   </gazebo>
   <gazebo reference="lidar_link">
-    <sensor name="gpu_lidar" type="gpu_lidar">
-      <update_rate>10</update_rate>
-      <topic>lidar</topic>
+    <sensor name="lidar_3d" type="gpu_lidar">
+      <always_on>true</always_on>
+      <update_rate>$(arg lidar_update_rate)</update_rate>
+      <topic>lidar_3d</topic>
       <gz_frame_id>lidar_link</gz_frame_id>
       <lidar>
         <scan>
           <horizontal>
-            <samples>360</samples>
+            <samples>$(arg lidar_horizontal_samples)</samples>
             <resolution>1</resolution>
             <min_angle>-3.14159</min_angle>
@@ -420,43 +399,13 @@
           </horizontal>
           <vertical>
-            <samples>1</samples>
+            <samples>$(arg lidar_vertical_samples)</samples>
             <resolution>1</resolution>
-            <min_angle>0</min_angle>
-            <max_angle>0</max_angle>
+            <min_angle>$(arg lidar_vertical_fov_min)</min_angle>
+            <max_angle>$(arg lidar_vertical_fov_max)</max_angle>
           </vertical>
         </scan>
         <range>
-          <min>0.2</min>
-          <max>20.0</max>
-        </range>
-      </lidar>
-      <always_on>true</always_on>
-      <visualize>true</visualize>
-    </sensor>
-  </gazebo>
-  <gazebo reference="lidar_3d_link">
-    <sensor name="lidar_3d" type="gpu_lidar">
-      <always_on>true</always_on>
-      <update_rate>10</update_rate>
-      <topic>lidar_3d</topic>
-      <gz_frame_id>lidar_3d_link</gz_frame_id>
-      <lidar>
-        <scan>
-          <horizontal>
-            <samples>360</samples>
-            <resolution>1</resolution>
-            <min_angle>-3.14159</min_angle>
-            <max_angle>3.14159</max_angle>
-          </horizontal>
-          <vertical>
-            <samples>16</samples>
-            <resolution>1</resolution>
-            <min_angle>-0.261799</min_angle>
-            <max_angle>0.261799</max_angle>
-          </vertical>
-        </scan>
-        <range>
-          <min>0.3</min>
-          <max>20.0</max>
+          <min>$(arg lidar_range_min)</min>
+          <max>$(arg lidar_range_max)</max>
         </range>
         <noise>

Commit message: help

File: src/exia_bringup/urdf/exia_ground.urdf.xacro (robot description, xacro)
@@ -316,4 +316,33 @@
     <child link="lidar_link"/>
     <origin xyz="0.3 0 0.42" rpy="0 0 0"/>
+  </joint>
+  <link name="gps_link">
+    <visual>
+      <origin xyz="0 0 0" rpy="0 0 0"/>
+      <geometry>
+        <box size="0.06 0.06 0.02"/>
+      </geometry>
+      <material name="white">
+        <color rgba="0.9 0.9 0.9 1"/>
+      </material>
+    </visual>
+    <collision>
+      <origin xyz="0 0 0" rpy="0 0 0"/>
+      <geometry>
+        <box size="0.06 0.06 0.02"/>
+      </geometry>
+    </collision>
+    <inertial>
+      <mass value="0.1"/>
+      <origin xyz="0 0 0" rpy="0 0 0"/>
+      <inertia ixx="0.00001" ixy="0" ixz="0"
+               iyy="0.00001" iyz="0"
+               izz="0.00001"/>
+    </inertial>
+  </link>
+  <joint name="gps_joint" type="fixed">
+    <parent link="base_link"/>
+    <child link="gps_link"/>
+    <origin xyz="0 0 0.35" rpy="0 0 0"/>
   </joint>
   <gazebo reference="front_left_wheel">
@@ -416,4 +445,42 @@
       </lidar>
       <visualize>true</visualize>
+    </sensor>
+  </gazebo>
+  <gazebo reference="gps_link">
+    <sensor name="navsat_sensor" type="navsat">
+      <always_on>true</always_on>
+      <update_rate>10</update_rate>
+      <topic>navsat</topic>
+      <gz_frame_id>gps_link</gz_frame_id>
+      <navsat>
+        <position_sensing>
+          <horizontal>
+            <noise type="gaussian">
+              <mean>0.0</mean>
+              <stddev>0.5</stddev>
+            </noise>
+          </horizontal>
+          <vertical>
+            <noise type="gaussian">
+              <mean>0.0</mean>
+              <stddev>1.0</stddev>
+            </noise>
+          </vertical>
+        </position_sensing>
+        <velocity_sensing>
+          <horizontal>
+            <noise type="gaussian">
+              <mean>0.0</mean>
+              <stddev>0.1</stddev>
+            </noise>
+          </horizontal>
+          <vertical>
+            <noise type="gaussian">
+              <mean>0.0</mean>
+              <stddev>0.1</stddev>
+            </noise>
+          </vertical>
+        </velocity_sensing>
+      </navsat>
     </sensor>
   </gazebo>

Commit message: help

File: src/exia_bringup/urdf/exia_ground.urdf.xacro (robot description, xacro)
@@ -316,4 +316,39 @@
     <child link="lidar_link"/>
     <origin xyz="0.3 0 0.42" rpy="0 0 0"/>
+  </joint>
+  <link name="camera_link">
+    <visual>
+      <origin xyz="0 0 0" rpy="0 0 0"/>
+      <geometry>
+        <box size="0.09 0.025 0.025"/>
+      </geometry>
+      <material name="dark_grey">
+        <color rgba="0.2 0.2 0.2 1"/>
+      </material>
+    </visual>
+    <collision>
+      <origin xyz="0 0 0" rpy="0 0 0"/>
+      <geometry>
+        <box size="0.09 0.025 0.025"/>
+      </geometry>
+    </collision>
+    <inertial>
+      <mass value="0.072"/>
+      <origin xyz="0 0 0" rpy="0 0 0"/>
+      <inertia ixx="0.00001" ixy="0" ixz="0"
+               iyy="0.00001" iyz="0"
+               izz="0.00001"/>
+    </inertial>
+  </link>
+  <joint name="camera_joint" type="fixed">
+    <parent link="base_link"/>
+    <child link="camera_link"/>
+    <origin xyz="0.4 0 0.52" rpy="0 0 0"/>
+  </joint>
+  <link name="camera_depth_optical_frame"/>
+  <joint name="camera_optical_joint" type="fixed">
+    <parent link="camera_link"/>
+    <child link="camera_depth_optical_frame"/>
+    <origin xyz="0 0 0" rpy="-1.5708 0 -1.5708"/>
   </joint>
   <link name="gps_link">
@@ -444,4 +479,35 @@
         </noise>
       </lidar>
+      <visualize>true</visualize>
+    </sensor>
+  </gazebo>
+  <gazebo reference="camera_link">
+    <sensor name="depth_camera" type="rgbd_camera">
+      <always_on>true</always_on>
+      <update_rate>15</update_rate>
+      <topic>depth_camera</topic>
+      <gz_frame_id>camera_depth_optical_frame</gz_frame_id>
+      <camera>
+        <horizontal_fov>1.7627</horizontal_fov>
+        <image>
+          <width>640</width>
+          <height>480</height>
+        </image>
+        <clip>
+          <near>0.2</near>
+          <far>20.0</far>
+        </clip>
+        <depth_camera>
+          <clip>
+            <near>0.2</near>
+            <far>20.0</far>
+          </clip>
+        </depth_camera>
+        <noise>
+          <type>gaussian</type>
+          <mean>0.0</mean>
+          <stddev>0.005</stddev>
+        </noise>
+      </camera>
       <visualize>true</visualize>
     </sensor>
